File: hardware/half-pint-turbidimeter_2.0.1.brd (EAGLE design)
At the start: 50.8 x 32 mm, 24 parts, among them IC1 MEGA8-AI

Commit message: minor edits to eagle schematics
Parts:
- moved FRAME1 5.00 mm to (18.9, -12.2)
Changed lines of the file:
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@@
 <?xml version="1.0" encoding="utf-8"?>
 <!DOCTYPE eagle SYSTEM "eagle.dtd">
-<eagle version="7.2.0">
+<eagle version="7.3.0">
 <drawing>
 <settings>
@@
 <attribute name="VALUE" x="38.1" y="25.781" size="0.4064" layer="25" font="vector"/>
 </element>
-<element name="FRAME1" library="SparkFun-Aesthetics" package="CREATIVE_COMMONS" value="FRAME-LETTER" x="20.955" y="-7.62"/>
+<element name="FRAME1" library="SparkFun-Aesthetics" package="CREATIVE_COMMONS" value="FRAME-LETTER" x="18.923" y="-12.192"/>
 <element name="C6" library="SparkFun" package="0603-CAP" value="100n" x="25.4" y="1.778" smashed="yes" rot="R180">
 <attribute name="VALUE" x="27.559" y="1.524" size="0.4064" layer="25" font="vector" rot="R90"/>
