File: hardware/half-pint-turbidimeter_led.brd (EAGLE design)
At the start: 6.6 x 18.8 mm, 3 parts

Commit message: minor edits to eagle schematics
Parts:
- added U$2: (no value), SparkFun-Aesthetics:CREATIVE_COMMONS
Other:
- board text added: "AWQUA"
Changed lines of the file:
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@@
 <hole x="3.302" y="17.526" drill="3"/>
 <hole x="3.302" y="3.302" drill="3"/>
+<text x="15.494" y="-7.366" size="1.778" layer="25">AWQUA</text>
 </plain>
 <attributes>
@@
 </element>
 <element name="U$1" library="awqua_eagle_library" package="AL5809" value="AL5809" x="4.826" y="9.144" rot="R180"/>
+<element name="U$2" library="SparkFun-Aesthetics" package="CREATIVE_COMMONS" value="" x="-14.986" y="-7.112"/>
 </elements>
 <signals>
