File: hardware/half-pint-turbidimeter_led.sch (EAGLE design)
At the start: 3 parts

Commit message: minor edits to eagle schematics
Parts:
- added FRAME1: FRAME-LETTER, SparkFun-Aesthetics:FRAME-LETTER
Other:
- note added: "AWQUA"
Changed lines of the file:
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@@
 <part name="D1" library="SparkFun-LED" deviceset="LED" device="5MM"/>
 <part name="U$1" library="awqua_eagle_library" deviceset="AL5809" device=""/>
+<part name="FRAME1" library="SparkFun-Aesthetics" deviceset="FRAME-LETTER" device=""/>
 </parts>
 <sheets>
 <sheet>
 <plain>
+<text x="139.7" y="17.78" size="2.54" layer="94">AWQUA</text>
 </plain>
 <instances>
@@
 <instance part="D1" gate="G$1" x="45.72" y="55.88" rot="R180"/>
 <instance part="U$1" gate="G$1" x="68.58" y="55.88" rot="R180"/>
+<instance part="FRAME1" gate="G$1" x="-27.94" y="7.62"/>
+<instance part="FRAME1" gate="V" x="119.38" y="7.62"/>
 </instances>
 <busses>
