File: hardware/half-pint-turbidimeter_tsl230rd_tsl267_1.0.1.brd (EAGLE design)
At the start: 12.7 x 15.2 mm, 8 parts

Commit message: hardware updates
Other:
- board text added: "awqua pocket turbidimeter tsl230rd / tsl267 brd v1.0.1 2016/03/14 github.com/awqua"
- board text removed: "awqua pocket turbidimeter tsl230rd / tsl267 brd v1.0 2016/03/14 github.com/awqua"
Changed lines of the file:
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@@
 pocket turbidimeter
 tsl230rd / tsl267 brd
-v1.0 2016/03/14
+v1.0.1 2016/03/14
 github.com/awqua</text>
 </plain>
@@
 <contactref element="C5" pad="2"/>
 <polygon width="0.254" layer="1">
-<vertex x="-3.556" y="42.926"/>
-<vertex x="50.292" y="43.18"/>
-<vertex x="50.8" y="-0.762"/>
+<vertex x="-2.794" y="17.272"/>
+<vertex x="17.272" y="17.272"/>
+<vertex x="17.018" y="-1.016"/>
 <vertex x="-3.048" y="-1.016"/>
 </polygon>
 <polygon width="0.254" layer="16">
-<vertex x="-2.54" y="43.434"/>
-<vertex x="50.038" y="44.196"/>
-<vertex x="50.292" y="-0.762"/>
-<vertex x="-2.54" y="-0.254"/>
+<vertex x="-1.778" y="18.034"/>
+<vertex x="18.034" y="18.288"/>
+<vertex x="17.526" y="-1.27"/>
+<vertex x="-2.794" y="-1.778"/>
 </polygon>
 <contactref element="JP1" pad="1"/>
